File: robot.sch (KiCad schematic (older format))
At the start: 15 parts, among them IC1 ATTINY2313-P, M1 CONN_5, M2 CONN_5, U1 ULN2003A, U2 ULN2003A

Commit message: Manufactured version
Connections:
- net GND: now also RPi1.25 (P24); no longer RPi1.26 (P22)
- net at IC1.2 ((RXD)PD0): now also RPi1.8 (P8); no longer RPi1.7 (P7)
- net at IC1.20 (VCC): now also RPi1.17 (P17); no longer RPi1.18 (P18)
- net at IC1.3 ((TXD)PD1): now also RPi1.10 (P10); no longer RPi1.9 (P9)
- net at R1.2: now also RPi1.19 (P19); no longer RPi1.20 (P20)
- net at R2.2: now also RPi1.21 (P21); no longer RPi1.22 (P22)
- net at R3.2: now also RPi1.23 (P23); no longer RPi1.24 (P20)
- net at R4.2: now also RPi1.15 (P15); no longer RPi1.16 (P16)
Changed lines of the file:
@@
-EESchema Schematic File Version 2  date Ut 23. jún 2015, 14:24:20 CEST
+EESchema Schematic File Version 2  date Ut 23. jún 2015, 16:40:48 CEST
 LIBS:power
 LIBS:device
@@
 Comment4 ""
 $EndDescr
-$Comp
-L CONN_13X2 RPi1
-U 1 1 55893BB7
-P 1200 2700
-F 0 "RPi1" H 1200 3400 60  0000 C CNN
-F 1 "CONN_13X2" V 1200 2700 50  0000 C CNN
-	1    1200 2700
-	1    0    0    1
-$EndComp
+Connection ~ 6850 1800
+Wire Wire Line
+	6850 1650 6850 3500
 Wire Wire Line
 	1600 2600 1650 2600
@@
 	3150 1150 4000 1150
 Wire Wire Line
-	3200 1450 3200 1300
-Wire Wire Line
-	3200 1300 2100 1300
-Wire Wire Line
 	2650 850  1800 850
 Wire Wire Line
@@
 Connection ~ 6850 2000
 Wire Wire Line
-	6100 3500 6850 3500
-Connection ~ 6850 1800
+	6850 3500 6100 3500
 Wire Wire Line
 	7400 3100 6400 3100
@@
 	4500 2000 3900 2000
 Wire Wire Line
-	1600 2500 2100 2500
-Wire Wire Line
 	1600 2300 1900 2300
 Connection ~ 4100 2000
@@
 	6500 3000 7400 3000
 Wire Wire Line
-	6850 3500 6850 1750
-Wire Wire Line
 	6850 3400 7400 3400
 Connection ~ 6850 3400
 Wire Wire Line
-	7400 2000 6850 2000
+	6850 2000 7400 2000
 Wire Wire Line
 	2500 2050 2350 2050
@@
 Wire Wire Line
 	4200 850  3150 850
-Wire Wire Line
-	2100 2500 2100 1300
 Wire Wire Line
 	2000 1150 2650 1150
@@
 Wire Wire Line
 	6850 1800 6100 1800
+Wire Wire Line
+	1600 2500 2100 2500
+Wire Wire Line
+	2100 2500 2100 1450
+Wire Wire Line
+	2100 1450 3200 1450
+$Comp
+L VCC #PWR?
+U 1 1 55896FEA
+P 6850 1650
+F 0 "#PWR?" H 6850 1750 30  0001 C CNN
+F 1 "VCC" H 6850 1750 30  0000 C CNN
+	1    6850 1650
+	1    0    0    -1
+$EndComp
+$Comp
+L CONN_13X2 RPi1
+U 1 1 55893BB7
+P 1200 2700
+F 0 "RPi1" H 1200 3400 60  0000 C CNN
+F 1 "CONN_13X2" V 1200 2700 50  0000 C CNN
+	1    1200 2700
+	-1   0    0    1
+$EndComp
 $Comp
 L R R4
@@
 	1    0    0    -1
 $EndComp
-$Comp
-L VCC #PWR2
-U 1 1 55891A39
-P 6850 1750
-F 0 "#PWR2" H 6850 1850 30  0001 C CNN
-F 1 "VCC" H 6850 1850 30  0000 C CNN
-	1    6850 1750
-	1    0    0    -1
-$EndComp
